Commit message: ㄱㄷㅈㄹㄷㄱㅁㅎㄱㄷㅎㄷㄱ

File: ros2/ASSY_URDF.SLDASM3/urdf/ASSY_URDF.SLDASM3.urdf (robot description, URDF)
Before this commit: robot ASSY_URDF.SLDASM2, 3 links, 2 joints
Links:
- link gripper_base: geometry collision mesh filename=package://ASSY_URDF.SLDASM3/meshes/gripper_base.STL; visual mesh filename=package://ASSY_URDF.SLDASM3/meshes/gripper_base.STL
- link gripper_joint_1: geometry collision mesh filename=package://ASSY_URDF.SLDASM3/meshes/gripper_joint_1.STL; visual mesh filename=package://ASSY_URDF.SLDASM3/meshes/gripper_joint_1.STL
- link gripper_joint_2: geometry collision mesh filename=package://ASSY_URDF.SLDASM3/meshes/gripper_joint_2.STL; visual mesh filename=package://ASSY_URDF.SLDASM3/meshes/gripper_joint_2.STL
Joints:
- joint gripper_joint_1_joint: axis 1 0 0 -> 0 0 -1; limit lower=0 upper=0.0525 effort=0 velocity=0 -> lower=0 upper=0 effort=0 velocity=0; origin xyz=0 -0.06 0.0525 rpy=1.5708 -1.5708 0 -> xyz=0 0.0525 0.06 rpy=1.5708 0 0
- joint gripper_joint_2_joint: axis 1 0 0 -> 0 0 -1; limit lower=0 upper=0.0525 effort=0 velocity=0 -> lower=0 upper=0 effort=0 velocity=0; origin xyz=0 -0.06 0.0145 rpy=1.5708 1.5708 0 -> xyz=0 -0.0525 0.06 rpy=-1.5708 0 0
