Commit message: urdf final

File: ros2/aidin_gripper_description/urdf/ASSY_URDF.SLDASM3.urdf (robot description, URDF)
Before this commit: robot ASSY_URDF.SLDASM3, 3 links, 2 joints
Joints:
- joint gripper_joint_1_joint: axis 0 0 -1 -> 0 0 1; limit lower=0 upper=0 effort=0 velocity=0 -> lower=0 upper=0.0525 effort=0 velocity=0
- joint gripper_joint_2_joint: axis 0 0 -1 -> 0 0 1; limit lower=0 upper=0 effort=0 velocity=0 -> lower=0 upper=0.0525 effort=0 velocity=0

Commit message: ros2 build settings

File: ros2/aidin_gripper_description/urdf/ASSY_URDF.SLDASM3.urdf (robot description, URDF)
Before this commit: robot ASSY_URDF.SLDASM3, 3 links, 2 joints
Links:
- link gripper_base: geometry collision mesh filename=package://aidin_gripper_description/meshes/gripper_base.STL; visual mesh filename=package://aidin_gripper_description/meshes/gripper_base.STL
- link gripper_joint_1: geometry collision mesh filename=package://aidin_gripper_description/meshes/gripper_joint_1.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; visual mesh filename=package://aidin_gripper_description/meshes/gripper_joint_1.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
- link gripper_joint_2: geometry collision mesh filename=package://aidin_gripper_description/meshes/gripper_joint_2.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; visual mesh filename=package://aidin_gripper_description/meshes/gripper_joint_2.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
